File: KiCAD5/FV01/FV-1.sch (KiCad schematic (older format))
At the start: 31 parts, among them J8 PROG, J9 SW_PROG, SW2 SW_EEPROM, U4 AE-FV-1-DIP_large, U5 24LC32, U6 74HC148

Commit message: Panel design
Parts:
- removed C22: 0.1u, Capacitor_THT:C_Rect_L7.0mm_W3.5mm_P5.00mm, symbol Device:C
- added C22: 1u, Capacitor_THT:CP_Radial_D5.0mm_P2.50mm, symbol Device:CP
- C16, C17, C19, C21: footprint Capacitor_THT:C_Rect_L7.0mm_W3.5mm_P5.00mm -> Capacitor_THT:C_Rect_L7.0mm_W2.5mm_P5.00mm
- RV3: renamed from RV5; footprint Potentiometer_THT:Potentiometer_Alps_RK09Y11_Single_Horizontal -> Potentiometer_THT:Potentiometer_Alps_RK097_Single_Horizontal
- RV4: renamed from RV6; footprint Potentiometer_THT:Potentiometer_Alps_RK09Y11_Single_Horizontal -> Potentiometer_THT:Potentiometer_Alps_RK097_Single_Horizontal
- RV5: renamed from RV7; footprint Potentiometer_THT:Potentiometer_Alps_RK09Y11_Single_Horizontal -> Potentiometer_THT:Potentiometer_Alps_RK097_Single_Horizontal
- renumbered J8 to J6, J9 to J7
Connections:
- net GND: now also J6.1 (Pin_1), J7.1 (Pin_1), C22.2; no longer J6.3 (Pin_3), J7.9 (Pin_9)
- net SCL: now also J6.3 (Pin_3); no longer J6.1 (Pin_1)
- net at U4.3 (MID): now also C22.1
- net at RN1.2 (R1), U6.4 (I7): now also J7.2 (Pin_2); no longer J7.8 (Pin_8)
- net at RN1.3 (R2), U6.3 (I6): now also J7.3 (Pin_3); no longer J7.7 (Pin_7)
- net at RN1.4 (R3), U6.2 (I5): now also J7.4 (Pin_4); no longer J7.6 (Pin_6)
- net at RN1.6 (R5), U6.13 (I3): now also J7.6 (Pin_6); no longer J7.4 (Pin_4)
- net at RN1.7 (R6), U6.12 (I2): now also J7.7 (Pin_7); no longer J7.3 (Pin_3)
- net at RN1.8 (R7), U6.11 (I1): now also J7.8 (Pin_8); no longer J7.2 (Pin_2)
- net at RN1.9 (R8), U6.10 (IO): now also J7.9 (Pin_9); no longer J7.1 (Pin_1)
