File: KiCAD5/FV01/FV01.sch (KiCad schematic (older format))
At the start: 49 parts, among them J1 ERK_PWR, J2 IN, J3 OUT, J6 TP_GND, J7 TP_GND, SW1 SW_MONO, U1 TL072, U2 TL072, U3 TA48M033F

Commit message: Panel design
Parts:
- removed J2: IN, Connector_JST:JST_XH_B4B-XH-A_1x04_P2.50mm_Vertical, symbol Connector_Generic:Conn_01x04
- removed RV1, RV3: 50k/A, Connector_PinHeader_2.54mm:PinHeader_1x03_P2.54mm_Vertical, symbol Device:R_POT
- removed RV2, RV4: 50k/B, Potentiometer_THT:Potentiometer_Alps_RK09Y11_Single_Horizontal, symbol Device:R_POT
- added J3: IN, Connector_JST:JST_XH_B4B-XH-A_1x04_P2.50mm_Vertical, symbol Connector_Generic:Conn_01x04
- added RV1: 50k/A, Potentiometer_THT:Potentiometer_Alps_RK097_Dual_Horizontal, symbol Device:R_POT_Dual_Separate
- added RV2: 50k/B, Potentiometer_THT:Potentiometer_Alps_RK097_Dual_Horizontal, symbol Device:R_POT_Dual_Separate
- C13: value 100u -> 100u OSCON
- renumbered C6 to C5, C5 to C6, J3 to J2, J6 to J4, J7 to J5, R9 to R8, R8 to R9
Connections:
- net FV-1/LFXIN: now also JP1.2; no longer SW1.2 (B)
- net FV-1/RFXIN: now also SW1.2 (B); no longer JP1.2
- net GND: now also J3.2 (Pin_2), J3.4 (Pin_4), RV1.1, RV1.4
- net LIN: now also J3.1 (Pin_1), RV1.3
- net RIN: now also J3.3 (Pin_3), RV1.6
- net at C3.2: now also RV1.2
- net at C1.1, JP1.1, R1.1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: now also RV2.1
- net at R5.2: now also RV2.2
- net at JP2.2: now also RV2.3
- net at C6.1, R7.1, SW1.3 (C)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: now also RV2.4
- net at R12.2: now also RV2.5
- net at C9.2: now also RV1.5
- net at JP3.2: now also RV2.6
Other:
- moved on the sheet: C1, C10, C2, C3, C4, C6, C8, C9, D3, J2, JP1, JP2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
